File: Scale_beta/Scale.sch (KiCad schematic (older format))
At the start: 16 parts, among them J1 Conn_01x04_Female, J2 Conn_01x03_Female, J3 Conn_01x07_Female, J4 Conn_01x07_Female, J5 Conn_01x07_Male

Commit message: Beta version
Parts:
- removed J3: Conn_01x07_Female, Connector_PinSocket_2.54mm:PinSocket_1x07_P2.54mm_Horizontal, symbol Connector:Conn_01x07_Female
- removed J5: Conn_01x07_Male, Connector_PinHeader_2.54mm:PinHeader_1x07_P2.54mm_Horizontal, symbol Connector:Conn_01x07_Male
Connections:
- net +5V: now also A3.28 (+5v)
- net GND: now also A3.25 (GND)
- net MISO: now also A3.19 (D10/MISO)
- net MOSI: now also A3.17 (D8/MOSI)
- net SCK: now also A3.18 (D9/SCK)
- net SS_ETH: now also A3.14 (D5/ETH_SS)
- net SS_SD: now also A3.13 (D4/SD_SS)
- net S renamed RELAY
Other:
- moved on the sheet: A1, A2, A3, H1, H2, H3, H4, H5, H6, H7, H8, J1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
